File: hardware/suspension_tension_meter.kicad_pcb (KiCad board)
At the start: 2 copper layers, 77 x 47 mm, 75 parts, among them J1 Conn_01x04, J2 Conn_01x06, J3 Conn_01x04, J4 Conn_01x04, J5 Terminator, SW1 Tactswitch, U1 STM32L4P5RET6, U2 AOZ1280CI, U3 LM1117-5.0, U4 LM1117-3.3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

Commit message: Port the project to KiCad 7
Other:
- rule pad_to_mask_clearance: 0 -> 0.05
