File: hardware/adc.kicad_sch (KiCad schematic)
At the start: 23 parts, among them U6 NAU7802SGI, U7 NAU7802SGI

Commit message: Release v1.0.0
Parts:
- renumbered C27 to C18, C25 to C19, C28 to C20, C23 to C21, C18 to C22, C19 to C23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
